File: temp_sense_redesign.kicad_sch (KiCad schematic)
At the start: 9 parts, among them IC1 TLV75533PDYDR, U2 AP63205

Commit message: Add files via upload
Parts:
- added C10, C11: 22p, Capacitor_SMD:C_1206_3216Metric_Pad1.33x1.80mm_HandSolder, symbol Device:C
- added C12: 0.1uF, Capacitor_SMD:C_1206_3216Metric_Pad1.33x1.80mm_HandSolder, symbol Device:C
- added C13, C16, C44: 1uF, Capacitor_SMD:C_0603_1608Metric, symbol Device:C_Small
- added C5: 10µ, symbol Device:C_Small
- added C6: 0.1µ, symbol Device:C_Small
- added C7: 100µ, symbol Device:C_Small
- added C8, C9: 0.1µ, Capacitor_SMD:C_1206_3216Metric_Pad1.33x1.80mm_HandSolder, symbol Device:C
- added R1: 47.5k, symbol Device:R_Small
- added R2: 120, symbol Device:R_Small
- added SW1: SW_Push, symbol Switch:SW_Push
- added U1: ~, symbol custom_components:MSPM0C1104SDGS20R
- added U3: MCP2517FDT-H_SL, symbol custom_components:MCP2517FDT-H_SL
- added U4: ~, symbol custom_components:TCAN1057A-Q1
- added U5, U6, U7: CLV4051ATDWRG4Q1, Package_SO:SOIC-16W_7.5x10.3mm_P1.27mm, symbol custom_components:CLV4051ATDWRG4Q1
- added Y1: Crystal, symbol Device:Crystal
- U2: footprint (none) -> Package_TO_SOT_SMD:TSOT-23-6
- renumbered C10 to C14, C11 to C15
Connections:
- net +3V3: now also C5.2, C6.2, R1.2, U1.6 (VDD); no longer C15.1, IC1.5 (OUT)
- net GND: now also C14.2, C10.2, C11.2, C12.1, C13.2, C16.2, C44.2, C5.1, C6.1, C7.2, C8.2, SW1.1, U1.7 (VSS), U3.7 (VSS), U4.2 (GND), U4.5 (S), U5.6 (Inh), U5.7 (VEE), U5.8 (VSS), U6.6 (Inh), U6.7 (VEE), U6.8 (VSS), U7.6 (Inh), U7.7 (VEE), U7.8 (VSS); no longer C14.1
- net at IC1.3 (EN): now also C14.1; no longer C14.2
- new net: C10.1, U3.6 (OSC1), Y1.1
- new net: U3.1 (TXCAN), U4.1 (TXD)
- new net: U3.2 (RXCAN), U4.4 (RXD)
- new net: C11.1, U3.5 (OSC2), Y1.2
- new net: C9.1, U4.3 (VCC)
- new net: C7.1, R1.1, SW1.2, U1.5 (PA1/NRST)
- new net +3.3V: C12.2, C13.1, C15.1, C16.1, C44.1, C8.1, IC1.5 (OUT), U3.14 (VDD), U4.8 (VIO), U5.16 (VDD), U6.16 (VDD), U7.16 (VDD)
- new net A: U1.8 (PA2), U5.11 (A), U6.11 (A), U7.11 (A)
- new net AI1: U1.20 (PA25/A2), U5.3 (X)
- new net AI2: U1.19 (PA24/A3), U6.3 (X), U7.3 (X)
- new net AI3: U1.17 (PA22/A4)
- new net AI4: U1.12 (PA16/A8)
- new net AI5: U1.1 (PA26/A1)
- new net B: U1.10 (PA6), U5.10 (B), U6.10 (B), U7.10 (B)
- new net C: U1.18 (PA23), U5.9 (C), U6.9 (C), U7.9 (C)
- new net CANL: R2.2, U4.7 (CANL)
- new net CAN_FD_INT: U1.9 (PA4), U3.4 (~{INT})
- new net CAN_H: R2.1, U4.6 (CANH)
- new net CS_CAN: U1.4 (PA0), U3.13 (NCS)
- new net SCK: U1.11 (PA11), U3.10 (SCK)
- new net SDI: U1.13 (PA17), U3.11 (SDI)
- new net SDO: U1.14 (PA18/A7), U3.12 (SDO)
- new net SWCLK: U1.16 (PA20/SWCLK)
- new net T1: U5.13 (X0)
- new net T10: U6.14 (X1)
- new net T11: U6.15 (X2)
- new net T12: U6.12 (X3)
- new net T13: U6.1 (X4)
- new net T14: U6.5 (X5)
- new net T15: U6.2 (X6)
- new net T16: U6.4 (X7)
- new net T17: U7.13 (X0)
- new net T18: U7.14 (X1)
- new net T19: U7.15 (X2)
- new net T2: U5.14 (X1)
- new net T20: U7.12 (X3)
- new net T21: U7.1 (X4)
- new net T22: U7.5 (X5)
- new net T23: U7.2 (X6)
- new net T24: U7.4 (X7)
- new net T3: U5.15 (X2)
- new net T4: U5.12 (X3)
- new net T5: U5.1 (X4)
- new net T6: U5.5 (X5)
- new net T7: U5.2 (X6)
- new net T8: U5.4 (X7)
- new net T9: U6.13 (X0)
- new net UART_RX: U1.3 (PA28/A5)
- new net UART_TX: U1.2 (PA27/A0)
- no-connect marks 0 -> 3
Other:
- moved on the sheet: C1, C14, C15, C2, C3, C4, IC1, L1, U2
